Commit message: model.sdf,model.sdf was updated by minho (2022.03.23)

File: rok3_model/urdf/rok3_model.urdf (robot description, URDF)
Before this commit: robot rok3_model, 16 links, 15 joints
Joints:
- joint L_Ankle_pitch_joint: origin xyz=0 0.0001 -0.35 rpy=0 0 0 -> xyz=0 -0.001 -0.35 rpy=0 0 0
- joint L_Foot_joint: origin xyz=0 0 -0.09 rpy=0 0 0 -> xyz=0 0.001 -0.09 rpy=0 0 0
- joint R_Ankle_pitch_joint: origin xyz=0 -0.0001 -0.35 rpy=0 0 0 -> xyz=0 0.001 -0.35 rpy=0 0 0
- joint R_Foot_joint: origin xyz=0 0 -0.09 rpy=0 0 0 -> xyz=0 -0.001 -0.09 rpy=0 0 0
